Commit message: unstable

File: unodopo_description/urdf/accessories/gazebo_diff_drive_plugin.xacro (robot description, xacro)
@@ -11,5 +11,5 @@
       <wheelSeparation>${wheel_separation}</wheelSeparation>
       <wheelDiameter>${wheel_radius * 2}</wheelDiameter>
-      <torque>30</torque>
+      <torque>20</torque>
       <commandTopic>cmd_vel</commandTopic>
       <odometryTopic>odom</odometryTopic>

File: unodopo_description/urdf/accessories/sick_scan.urdf.xacro (robot description, xacro)
@@ -4,7 +4,7 @@
   xmlns:sensor="http://playerstage.sourceforge.net/gazebo/xmlschema/#sensor"
   xmlns:xacro="http://ros.org/wiki/xacro">
-  <xacro:macro name="sick_tim_57x" params="wheel_offset name ros_topic min_angle:=-2.357 max_angle:=2.357 gaussian_noise:=0.01 samples:=811">
+  <xacro:macro name="sick_tim_57x" params="wheel_offset name ros_topic visualize min_angle:=-2.357 max_angle:=2.357 gaussian_noise:=0.01 samples:=811">
     <xacro:sick_tim name="${name}" ros_topic="${ros_topic}"
-      length="0.06" width="0.06" height="0.079" mass="0.150" z_offset="0.05595"
+      length="0.06" width="0.06" height="0.079" mass="0.150" z_offset="0.05595" visualize="${visualize}"
       min_angle="${min_angle}" max_angle="${max_angle}"
       min_range="0.05" max_range="25.0" gaussian_noise="${gaussian_noise}" samples="${samples}"
@@ -13,5 +13,5 @@
       wheel_offset="${wheel_offset}" /> <!-- edited for unodopo-->
   </xacro:macro>
-  <xacro:macro name="sick_tim" params="name ros_topic length width height mass z_offset min_angle max_angle min_range max_range gaussian_noise samples mesh scale wheel_offset">
+  <xacro:macro name="sick_tim" params="name ros_topic length width height mass z_offset visualize min_angle max_angle min_range max_range gaussian_noise samples mesh scale wheel_offset">
     <!-- z_offset: distance between base plate and laser center (= center of mesh) -->
     <joint name="{name}_mount_joint" type="fixed">
@@ -58,7 +58,7 @@
       </inertial>
     </link>
-    <xacro:sick_tim_laser_gazebo_v0 name="${name}" link="${name}" ros_topic="${ros_topic}" update_rate="15.0" min_angle="${min_angle}" max_angle="${max_angle}" min_range="${min_range}" max_range="${max_range}" gaussian_noise="${gaussian_noise}" samples="${samples}" />
+    <xacro:sick_tim_laser_gazebo_v0 name="${name}" link="${name}" ros_topic="${ros_topic}" update_rate="15.0" visualize="${visualize}" min_angle="${min_angle}" max_angle="${max_angle}" min_range="${min_range}" max_range="${max_range}" gaussian_noise="${gaussian_noise}" samples="${samples}" />
   </xacro:macro>
-  <xacro:macro name="sick_tim_laser_gazebo_v0" params="name link ros_topic update_rate min_angle max_angle min_range max_range gaussian_noise samples">
+  <xacro:macro name="sick_tim_laser_gazebo_v0" params="name link ros_topic update_rate visualize min_angle max_angle min_range max_range gaussian_noise samples">
     <gazebo reference="${link}">
       <material value="Gazebo/Blue" />
@@ -67,5 +67,5 @@
         <update_rate>${update_rate}</update_rate>
         <pose>0 0 0 0 0 0</pose>
-        <visualize>true</visualize>
+        <visualize>${visualize}</visualize>
         <ray>
           <scan>

File: unodopo_description/urdf/unodopo.urdf (robot description, URDF)
Before this commit: robot unodopo, 11 links, 10 joints
Links:
- added link base_footprint
Joints:
- added joint base_joint: type fixed, parent base_footprint, child base_link, origin xyz=0 0 -${wheel_offset} rpy=0 0 0
