Commit message: unodopo not jumpy anymore

File: unodopo_description/urdf/accessories/sick_scan.urdf.xacro (robot description, xacro)
@@ -1,4 +1,4 @@
 <?xml version="1.0"?>
-<robot name="laser" xmlns:controller="http://playerstage.sourceforge.net/gazebo/xmlschema/#controller"
+<robot xmlns:controller="http://playerstage.sourceforge.net/gazebo/xmlschema/#controller"
   xmlns:interface="http://playerstage.sourceforge.net/gazebo/xmlschema/#interface"
   xmlns:sensor="http://playerstage.sourceforge.net/gazebo/xmlschema/#sensor"
@@ -9,5 +9,5 @@
       min_angle="${min_angle}" max_angle="${max_angle}"
       min_range="0.05" max_range="25.0" gaussian_noise="${gaussian_noise}" samples="${samples}"
-      mesh="package://unodopo/meshes/accessories/sick_tim_5xx.stl"
+      mesh="package://unodopo/meshes/accessories/sick_tim571.stl"
       scale="0.001 0.001 0.001"
       wheel_offset="${wheel_offset}" /> <!-- edited for unodopo-->
@@ -18,17 +18,13 @@
       <parent link="base_link"/>
       <child link="${name}_mount_link"/>
-      <origin xyz="0 0 0"/>
+      <origin xyz="-0.2775 0 0.320"/>
     </joint>
+    <!-- note that in this case, mount_link is actually not necessary since I made the origin of the lidar to be offset already in the STL file-->
     <link name="${name}_mount_link">
-      <inertial>
-        <mass value="0.001" />
-        <origin xyz="0 0 -${wheel_offset}"/>
-        <inertia ixx="0.000001" ixy="0.0" ixz="0.0"
-          iyy="0.000001" iyz="0.0" izz="0.000001" />
-      </inertial>
       <visual>
         <geometry>
-          <mesh filename="${mesh} ${scale}" />
+          <mesh filename="${mesh}" scale="${scale}" />
         </geometry>
+        <origin xyz="0 0 0"/>
         <material name="blue" >
           <color rgba="0 0 1 1" />
@@ -37,30 +33,24 @@
       <collision>
         <geometry>
-          <mesh filename="${mesh} ${scale}" />
+          <mesh filename="${mesh}" scale="${scale}" />
         </geometry>
+        <origin xyz="0 0 0"/>
       </collision>
+      <inertial>
+        <mass value="0.001" />
+        <origin xyz="0 0 0"/>
+        <inertia ixx="0.000001" ixy="0.0" ixz="0.0"
+          iyy="0.000001" iyz="0.0" izz="0.000001" />
+      </inertial>
     </link>
     <joint name="${name}_joint" type="fixed">
       <parent link="${name}_mount_link" />
       <child link="${name}" />
-      <origin rpy="0 0 0" xyz="0 0 ${z_offset}"/>
+      <origin xyz="0 0 0" rpy="0 0 ${pi}"/>
     </joint>
     <link name="${name}">
-      <visual>
-        <geometry>
-          <mesh filename="${mesh} ${scale}" />
-        </geometry>
-        <material name="blue" >
-          <color rgba="0 0 1 1" />
-        </material>
-      </visual>
-      <collision>
-        <geometry>
-          <mesh filename="${mesh} ${scale}" />
-        </geometry>
-      </collision>
       <inertial>
         <mass value="${mass}" />
-        <origin xyz="0 0 -0.026" />
+        <origin xyz="0 0 0" rpy="0 0 0"/>
         <inertia ixx="${0.0833333 * mass * (width * width + height * height)}" ixy="0.0" ixz="0.0"
           iyy="${0.0833333 * mass * (length * length + height * height)}" iyz="0.0"
@@ -77,5 +67,5 @@
         <update_rate>${update_rate}</update_rate>
         <pose>0 0 0 0 0 0</pose>
-        <visualize>false</visualize>
+        <visualize>true</visualize>
         <ray>
           <scan>

File: unodopo_description/urdf/unodopo.urdf (robot description, URDF)
Before this commit: robot unodopo, 11 links, 10 joints
Links:
- link caster_mount_backleft: geometry collision sphere radius=0.005; visual mesh filename=package://unodopo/meshes/accessories/caster_mount_backleft.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 scale=0.001 0.001 0.001
- link caster_mount_backright: geometry collision sphere radius=0.005; visual mesh filename=package://unodopo/meshes/accessories/caster_mount_backright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 scale=0.001 0.001 0.001
- link caster_mount_frontleft: geometry collision sphere radius=0.005; visual mesh filename=package://unodopo/meshes/accessories/caster_mount_frontleft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 scale=0.001 0.001 0.001
- link caster_mount_frontright: geometry collision sphere radius=0.005; visual mesh filename=package://unodopo/meshes/accessories/caster_mount_frontrigh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 scale=0.001 0.001 0.001
- link caster_wheel_backleft: geometry collision cylinder length=0.02 radius=0.02; visual mesh filename=package://unodopo/meshes/accessories/caster_wheel_backleft.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 scale=0.001 0.001 0.001
- link caster_wheel_backright: geometry collision cylinder length=0.02 radius=0.02; visual mesh filename=package://unodopo/meshes/accessories/caster_wheel_backright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 scale=0.001 0.001 0.001
- link caster_wheel_frontleft: geometry collision cylinder length=0.02 radius=0.02; visual mesh filename=package://unodopo/meshes/accessories/caster_wheel_frontleft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 scale=0.001 0.001 0.001
- link caster_wheel_frontright: geometry collision cylinder length=0.02 radius=0.02; visual mesh filename=package://unodopo/meshes/accessories/caster_wheel_frontrigh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 scale=0.001 0.001 0.001
Joints:
- joint right_wheel_joint: origin xyz=0 0 0 -> xyz=0 0 0.01

Commit message: corrected CMakeLists and  finally stable in gazebo

File: unodopo_description/urdf/accessories/sick_scan.urdf.xacro (robot description, xacro)
@@ -9,5 +9,5 @@
       min_angle="${min_angle}" max_angle="${max_angle}"
       min_range="0.05" max_range="25.0" gaussian_noise="${gaussian_noise}" samples="${samples}"
-      mesh="package://unodopo/meshes/accessories/sick_tim571.stl"
+      mesh="package://unodopo_description/meshes/accessories/sick_tim571.stl"
       scale="0.001 0.001 0.001"
       wheel_offset="${wheel_offset}" /> <!-- edited for unodopo-->

File: unodopo_description/urdf/unodopo.urdf (robot description, URDF)
Before this commit: robot unodopo, 12 links, 11 joints
Links:
- link base_link: geometry collision mesh filename=package://unodopo_description/meshes/unodopo_main_body.stl scale=0.001 0.001 0.001; visual mesh filename=package://unodopo_description/meshes/unodopo_main_body.stl scale=0.001 0.001 0.001
- link caster_mount_backleft: geometry collision sphere radius=0.005; visual mesh filename=package://unodopo_description/meshes/accessories/caster_mou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 scale=0.001 0.001 0.001
- link caster_mount_backright: geometry collision sphere radius=0.005; visual mesh filename=package://unodopo_description/meshes/accessories/caster_mou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 scale=0.001 0.001 0.001
- link caster_mount_frontleft: geometry collision sphere radius=0.005; visual mesh filename=package://unodopo_description/meshes/accessories/caster_mou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 scale=0.001 0.001 0.001
- link caster_mount_frontright: geometry collision sphere radius=0.005; visual mesh filename=package://unodopo_description/meshes/accessories/caster_mou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 scale=0.001 0.001 0.001
- link caster_wheel_backleft: geometry collision cylinder length=0.02 radius=0.02; visual mesh filename=package://unodopo_description/meshes/accessories/caster_whe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 scale=0.001 0.001 0.001
- link caster_wheel_backright: geometry collision cylinder length=0.02 radius=0.02; visual mesh filename=package://unodopo_description/meshes/accessories/caster_whe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 scale=0.001 0.001 0.001
- link caster_wheel_frontleft: geometry collision cylinder length=0.02 radius=0.02; visual mesh filename=package://unodopo_description/meshes/accessories/caster_whe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 scale=0.001 0.001 0.001
- link caster_wheel_frontright: geometry collision cylinder length=0.02 radius=0.02; visual mesh filename=package://unodopo_description/meshes/accessories/caster_whe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 scale=0.001 0.001 0.001
- link left_wheel: geometry collision mesh filename=package://unodopo_description/meshes/unodopo_left_wheel.stl scale=0.001 0.001 0.001; visual mesh filename=package://unodopo_description/meshes/unodopo_left_wheel.stl scale=0.001 0.001 0.001
- link right_wheel: geometry collision mesh filename=package://unodopo_description/meshes/unodopo_right_wheel.stl scale=0.001 0.001 0.001; visual mesh filename=package://unodopo_description/meshes/unodopo_right_wheel.stl scale=0.001 0.001 0.001
Joints:
- joint caster_wheel_backleft_joint: origin xyz=0.014874 0 ${-0.07465+wheel_offset} -> xyz=0.014 0 ${-0.069+wheel_offset}
- joint caster_wheel_backright_joint: origin xyz=0.014874 0 ${-0.07465+wheel_offset} -> xyz=0.014 0 ${-0.069+wheel_offset}
- joint caster_wheel_frontleft_joint: origin xyz=0.014874 0 ${-0.07465+wheel_offset} -> xyz=0.014 0 ${-0.069+wheel_offset}
- joint caster_wheel_frontright_joint: origin xyz=0.014874 0 ${-0.07465+wheel_offset} -> xyz=0.014 0 ${-0.069+wheel_offset}
- joint left_wheel_joint: origin xyz=0 0 0 -> xyz=0 0 0.01
