Commit message: for abi to check

File: unodopo_description/urdf/unodopo.urdf (robot description, URDF)
Before this commit: robot unodopo, 3 links, 2 joints
Links:
- added link caster_mount_backleft, mass 0.1; collision mesh filename=package://unodopo/meshes/accessories/caster_mount_backleft.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 scale=0.001 0.001 0.001; visual mesh filename=package://unodopo/meshes/accessories/caster_mount_backleft.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 scale=0.001 0.001 0.001
- added link caster_mount_backright, mass 0.1; collision mesh filename=package://unodopo/meshes/accessories/caster_mount_backright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 scale=0.001 0.001 0.001; visual mesh filename=package://unodopo/meshes/accessories/caster_mount_backright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 scale=0.001 0.001 0.001
- added link caster_mount_frontleft, mass 0.1; collision mesh filename=package://unodopo/meshes/accessories/caster_mount_frontleft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 scale=0.001 0.001 0.001; visual mesh filename=package://unodopo/meshes/accessories/caster_mount_frontleft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 scale=0.001 0.001 0.001
- added link caster_mount_frontright, mass 0.1; collision mesh filename=package://unodopo/meshes/accessories/caster_mount_frontrigh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 scale=0.001 0.001 0.001; visual mesh filename=package://unodopo/meshes/accessories/caster_mount_frontrigh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 scale=0.001 0.001 0.001
- added link caster_wheel_backleft, mass ${caster_wheel_mass}; collision mesh filename=package://unodopo/meshes/accessories/caster_wheel_backleft.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 scale=0.001 0.001 0.001; visual mesh filename=package://unodopo/meshes/accessories/caster_wheel_backleft.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 scale=0.001 0.001 0.001
- added link caster_wheel_backright, mass ${caster_wheel_mass}; collision mesh filename=package://unodopo/meshes/accessories/caster_wheel_backright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 scale=0.001 0.001 0.001; visual mesh filename=package://unodopo/meshes/accessories/caster_wheel_backright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 scale=0.001 0.001 0.001
- added link caster_wheel_frontleft, mass ${caster_wheel_mass}; collision mesh filename=package://unodopo/meshes/accessories/caster_wheel_frontleft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 scale=0.001 0.001 0.001; visual mesh filename=package://unodopo/meshes/accessories/caster_wheel_frontleft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 scale=0.001 0.001 0.001
- added link caster_wheel_frontright, mass ${caster_wheel_mass}; collision mesh filename=package://unodopo/meshes/accessories/caster_wheel_frontrigh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 scale=0.001 0.001 0.001; visual mesh filename=package://unodopo/meshes/accessories/caster_wheel_frontrigh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 scale=0.001 0.001 0.001
- link base_link: geometry collision mesh filename=package://unodopo/meshes/unodopo_main_body.stl scale=0.001 0.001 0.001; visual mesh filename=package://unodopo/meshes/unodopo_main_body.stl scale=0.001 0.001 0.001
Joints:
- added joint caster_mount_backleft_joint: type continuous, parent base_link, child caster_mount_backleft, origin xyz=0.210 -0.120 -0.040, axis 0 0 1
- added joint caster_mount_backright_joint: type continuous, parent base_link, child caster_mount_backright, origin xyz=0.210 0.120 -0.040, axis 0 0 1
- added joint caster_mount_frontleft_joint: type continuous, parent base_link, child caster_mount_frontleft, origin xyz=-0.210 -0.120 -0.040, axis 0 0 1
- added joint caster_mount_frontright_joint: type continuous, parent base_link, child caster_mount_frontright, origin xyz=-0.210 0.120 -0.040, axis 0 0 1
- added joint caster_wheel_backleft_joint: type continuous, parent caster_mount_backleft, child caster_wheel_backleft, origin xyz=0.014874 0 ${-0.07465+wheel_offset}, axis 0 1 0
- added joint caster_wheel_backright_joint: type continuous, parent caster_mount_backright, child caster_wheel_backright, origin xyz=0.014874 0 ${-0.07465+wheel_offset}, axis 0 1 0
- added joint caster_wheel_frontleft_joint: type continuous, parent caster_mount_frontleft, child caster_wheel_frontleft, origin xyz=0.014874 0 ${-0.07465+wheel_offset}, axis 0 1 0
- added joint caster_wheel_frontright_joint: type continuous, parent caster_mount_frontright, child caster_wheel_frontright, origin xyz=0.014874 0 ${-0.07465+wheel_offset}, axis 0 1 0

Commit message: updated urdf

File: unodopo_description/urdf/unodopo.urdf (robot description, URDF)
Before this commit: robot unodopo, 12 links, 11 joints
Links:
- link caster_wheel_backleft: geometry collision cylinder length=0.02 radius=0.025; visual mesh filename=package://unodopo_description/meshes/accessories/caster_whe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 scale=0.001 0.001 0.001
- link caster_wheel_backright: geometry collision cylinder length=0.02 radius=0.025; visual mesh filename=package://unodopo_description/meshes/accessories/caster_whe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 scale=0.001 0.001 0.001
- link caster_wheel_frontleft: geometry collision cylinder length=0.02 radius=0.025; visual mesh filename=package://unodopo_description/meshes/accessories/caster_whe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 scale=0.001 0.001 0.001
- link caster_wheel_frontright: geometry collision cylinder length=0.02 radius=0.025; visual mesh filename=package://unodopo_description/meshes/accessories/caster_whe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 scale=0.001 0.001 0.001
Joints:
- joint base_joint: child base_link -> base_footprint; parent base_footprint -> base_link
- joint left_wheel_joint: origin xyz=0 0 0.01 -> xyz=0 0 0.004
- joint right_wheel_joint: origin xyz=0 0 0.01 -> xyz=0 0 0.004
